File: ControllerPCB/ControllerPCB.kicad_pcb (KiCad board)
At the start: 2 copper layers, 220 x 125 mm, 26 parts, among them J1 Conn_01x02_Male, J10 Conn_01x06_Male, J11 Conn_01x02_Male, J12 Conn_01x02_Male, J2 Conn_01x04_Male, J3 Conn_01x02_Male, J4 Conn_01x03_Male, J5 Conn_01x03_Male, J6 Conn_01x02_Male, J7 A-2004-2-4-LPS-N-R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

Commit message: Fix Typo in Spooler
Other:
- board text added: "Spooler"
- board text removed: "Spoiler"
