File: PCB/Controller/ControllerPCB.sch (KiCad schematic (older format))
At the start: 26 parts, among them J1 Conn_01x02_Male, J10 Conn_01x06_Male, J11 Conn_01x02_Male, J12 Conn_01x02_Male, J2 Conn_01x04_Male, J3 Conn_01x02_Male, J4 Conn_01x03_Male, J5 Conn_01x03_Male, J6 Conn_01x02_Male, J7 A-2004-2-4-LPS-N-R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

Commit message: Schematic now fits on a letter size page.  Output to PDF.
Other:
- note added: "I2C Pullup"
- note added: "Roller Motor"
- note added: "Screw Motor"
- note added: "Slack Sensor"
- note added: "Spooler Motor"
- note removed: "Pullup Resistors for I2c"
- note removed: "Roller Motor Output"
- note removed: "ScrewMotor"
- note removed: "SlackSensor"
- note removed: "SpollerMotor"
- moved on the sheet: D1, D2, D3, D4, J1, J10, J11, J12, J2, J3, J4, J5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

Commit message: Updated controller PCB.
Parts:
- D1, D2, D3, D4: symbol Device:D -> ControllerPCB-rescue:D-Device-ControllerPCB-rescue
- J1, J11, J12, J3, J6: symbol Connector:Conn_01x02_Male -> ControllerPCB-rescue:Conn_01x02_Male-Connector-ControllerPCB-rescue
- J10: symbol Connector:Conn_01x06_Male -> ControllerPCB-rescue:Conn_01x06_Male-Connector-ControllerPCB-rescue
- J2, J8, J9: symbol Connector:Conn_01x04_Male -> ControllerPCB-rescue:Conn_01x04_Male-Connector-ControllerPCB-rescue
- J4, J5: symbol Connector:Conn_01x03_Male -> ControllerPCB-rescue:Conn_01x03_Male-Connector-ControllerPCB-rescue
- Q1, Q2: symbol Transistor_FET:2N7002 -> ControllerPCB-rescue:2N7002-Transistor_FET-ControllerPCB-rescue
- R1, R2, R3, R4: symbol Device:R -> ControllerPCB-rescue:R-Device-ControllerPCB-rescue
Changed lines of the file:
@@
 $EndComp
 $Comp
-L power:GND #PWR027
+L ControllerPCB-rescue:GND-power-ControllerPCB-rescue #PWR027
 U 1 1 605B261D
 P 10150 4150
@@
 	10300 3450 9950 3450
 $Comp
-L power:GND #PWR022
+L ControllerPCB-rescue:GND-power-ControllerPCB-rescue #PWR022
 U 1 1 605B48B7
 P 7050 2350
@@
 	7200 2350 7350 2350
 $Comp
-L power:+3.3V #PWR05
+L ControllerPCB-rescue:+3.3V-power-ControllerPCB-rescue #PWR05
 U 1 1 605B5E31
 P 1000 5000
@@
 	1000 5000 1150 5000
 $Comp
-L power:GND #PWR03
+L ControllerPCB-rescue:GND-power-ControllerPCB-rescue #PWR03
 U 1 1 605B64CE
 P 850 4500
@@
 $EndComp
 $Comp
-L power:GND #PWR023
+L ControllerPCB-rescue:GND-power-ControllerPCB-rescue #PWR023
 U 1 1 605B8B46
 P 8150 3400
@@
 SCL
 $Comp
-L Transistor_FET:2N7002 Q2
+L ControllerPCB-rescue:2N7002-Transistor_FET-ControllerPCB-rescue Q2
 U 1 1 605BDF2C
 P 9900 6000
@@
 $EndComp
 $Comp
-L power:GND #PWR026
+L ControllerPCB-rescue:GND-power-ControllerPCB-rescue #PWR026
 U 1 1 605C74D4
 P 10000 6350
@@
 $EndComp
 $Comp
-L Device:R R4
+L ControllerPCB-rescue:R-Device-ControllerPCB-rescue R4
 U 1 1 605CADF4
 P 9700 6200
@@
 I2C Pullup
 $Comp
-L Device:R R1
+L ControllerPCB-rescue:R-Device-ControllerPCB-rescue R1
 U 1 1 605D250C
 P 3650 6400
@@
 $EndComp
 $Comp
-L Device:R R2
+L ControllerPCB-rescue:R-Device-ControllerPCB-rescue R2
 U 1 1 605D268F
 P 3950 6400
@@
 SCL
 $Comp
-L Connector:Conn_01x06_Male J10
+L ControllerPCB-rescue:Conn_01x06_Male-Connector-ControllerPCB-rescue J10
 U 1 1 605D514E
 P 7600 5700
@@
 RollerMotor-
 $Comp
-L power:GND #PWR025
+L ControllerPCB-rescue:GND-power-ControllerPCB-rescue #PWR025
 U 1 1 605D7349
 P 8650 5700
@@
 Slack Sensor
 $Comp
-L Connector:Conn_01x04_Male J2
+L ControllerPCB-rescue:Conn_01x04_Male-Connector-ControllerPCB-rescue J2
 U 1 1 605EB896
 P 2150 7500
@@
 $EndComp
 $Comp
-L power:GND #PWR07
+L ControllerPCB-rescue:GND-power-ControllerPCB-rescue #PWR07
 U 1 1 605EC293
 P 2900 7400
@@
 Tachometer
 $Comp
-L Connector:Conn_01x03_Male J5
+L ControllerPCB-rescue:Conn_01x03_Male-Connector-ControllerPCB-rescue J5
 U 1 1 605F2464
 P 5100 6250
@@
 $EndComp
 $Comp
-L power:GND #PWR015
+L ControllerPCB-rescue:GND-power-ControllerPCB-rescue #PWR015
 U 1 1 605F295E
 P 5700 6400
@@
 Scales
 $Comp
-L Connector:Conn_01x02_Male J1
+L ControllerPCB-rescue:Conn_01x02_Male-Connector-ControllerPCB-rescue J1
 U 1 1 605FC928
 P 3750 7450
@@
 $EndComp
 $Comp
-L Connector:Conn_01x02_Male J3
+L ControllerPCB-rescue:Conn_01x02_Male-Connector-ControllerPCB-rescue J3
 U 1 1 605FCF26
 P 5250 7450
@@
 $EndComp
 $Comp
-L power:GND #PWR02
+L ControllerPCB-rescue:GND-power-ControllerPCB-rescue #PWR02
 U 1 1 605FD458
 P 4200 7450
@@
 	4200 7450 3950 7450
 $Comp
-L power:GND #PWR08
+L ControllerPCB-rescue:GND-power-ControllerPCB-rescue #PWR08
 U 1 1 605FEF03
 P 5800 7500
@@
 SpollerMotor
 $Comp
-L Transistor_FET:2N7002 Q1
+L ControllerPCB-rescue:2N7002-Transistor_FET-ControllerPCB-rescue Q1
 U 1 1 6060B486
 P 6200 3750
@@
 $EndComp
 $Comp
-L power:GND #PWR017
+L ControllerPCB-rescue:GND-power-ControllerPCB-rescue #PWR017
 U 1 1 6060B48C
 P 6300 4100
@@
 $EndComp
 $Comp
-L Device:R R3
+L ControllerPCB-rescue:R-Device-ControllerPCB-rescue R3
 U 1 1 6060B493
 P 6000 3950
@@
 	6200 3200 6300 3200
 $Comp
-L Connector:Conn_01x02_Male J6
+L ControllerPCB-rescue:Conn_01x02_Male-Connector-ControllerPCB-rescue J6
 U 1 1 606176F7
 P 4800 3900
@@
 Fans-
 $Comp
-L Connector:Conn_01x04_Male J8
+L ControllerPCB-rescue:Conn_01x04_Male-Connector-ControllerPCB-rescue J8
 U 1 1 60618AAD
 P 850 6400
@@
 $EndComp
 $Comp
-L Connector:Conn_01x04_Male J9
+L ControllerPCB-rescue:Conn_01x04_Male-Connector-ControllerPCB-rescue J9
 U 1 1 6061ADD1
 P 1950 6400
@@
 ScaleCLK2
 $Comp
-L power:+5V #PWR018
+L ControllerPCB-rescue:+5V-power-ControllerPCB-rescue #PWR018
 U 1 1 6061D833
 P 1350 6750
@@
 $EndComp
 $Comp
-L power:+5V #PWR019
+L ControllerPCB-rescue:+5V-power-ControllerPCB-rescue #PWR019
 U 1 1 6061DEAF
 P 2550 6750
@@
 $EndComp
 $Comp
-L power:GND #PWR09
+L ControllerPCB-rescue:GND-power-ControllerPCB-rescue #PWR09
 U 1 1 60626B47
 P 4850 2000
@@
 	4850 2000 5150 2000
 $Comp
-L power:GND #PWR011
+L ControllerPCB-rescue:GND-power-ControllerPCB-rescue #PWR011
 U 1 1 6062ADC7
 P 4900 1400
@@
 SCL
 $Comp
-L power:GND #PWR012
+L ControllerPCB-rescue:GND-power-ControllerPCB-rescue #PWR012
 U 1 1 6062EBC7
 P 1650 7550
@@
 	1500 7550 1650 7550
 $Comp
-L power:+5V #PWR029
+L ControllerPCB-rescue:+5V-power-ControllerPCB-rescue #PWR029
 U 1 1 60636D5E
 P 10300 3450
@@
 $EndComp
 $Comp
-L power:+5V #PWR0101
+L ControllerPCB-rescue:+5V-power-ControllerPCB-rescue #PWR0101
 U 1 1 605E7A4C
 P 3800 6150
@@
 	7800 5700 8650 5700
 $Comp
-L power:+5V #PWR024
+L ControllerPCB-rescue:+5V-power-ControllerPCB-rescue #PWR024
 U 1 1 605D9A42
 P 8900 6000
@@
 	8450 6000 8900 6000
 $Comp
-L power:+5V #PWR0102
+L ControllerPCB-rescue:+5V-power-ControllerPCB-rescue #PWR0102
 U 1 1 6062089A
 P 8150 5500
@@
 Vin
 $Comp
-L Connector:Conn_01x03_Male J4
+L ControllerPCB-rescue:Conn_01x03_Male-Connector-ControllerPCB-rescue J4
 U 1 1 60628487
 P 1300 7450
@@
 Vin
 $Comp
-L Connector:Conn_01x02_Male J12
+L ControllerPCB-rescue:Conn_01x02_Male-Connector-ControllerPCB-rescue J12
 U 1 1 6062B5BD
 P 4750 3500
@@
 Fans-
 $Comp
-L Connector:Conn_01x02_Male J11
+L ControllerPCB-rescue:Conn_01x02_Male-Connector-ControllerPCB-rescue J11
 U 1 1 6062F882
 P 4750 3100
@@
 	6300 2900 6250 2900
 $Comp
-L Device:D D1
+L ControllerPCB-rescue:D-Device-ControllerPCB-rescue D1
 U 1 1 6066CFE2
 P 6300 3350
@@
 	6300 3500 6300 3550
 $Comp
-L Device:D D4
+L ControllerPCB-rescue:D-Device-ControllerPCB-rescue D4
 U 1 1 60675D3C
 P 6300 3050
@@
 $EndComp
 $Comp
-L Device:D D3
+L ControllerPCB-rescue:D-Device-ControllerPCB-rescue D3
 U 1 1 606853B4
 P 10000 5150
@@
 $EndComp
 $Comp
-L Device:D D2
+L ControllerPCB-rescue:D-Device-ControllerPCB-rescue D2
 U 1 1 606864CA
 P 10000 5600
@@
 LV2
 $Comp
-L power:+5V #PWR0103
+L ControllerPCB-rescue:+5V-power-ControllerPCB-rescue #PWR0103
 U 1 1 606BA9A1
 P 5700 6150
@@
 $EndComp
 $Comp
-L power:+5V #PWR0104
+L ControllerPCB-rescue:+5V-power-ControllerPCB-rescue #PWR0104
 U 1 1 606BC1EC
 P 3100 7700
@@
 Vin
 $Comp
-L power:+5V #PWR0105
+L ControllerPCB-rescue:+5V-power-ControllerPCB-rescue #PWR0105
 U 1 1 6063DDF5
 P 750 5100
