File: Wiring/ValpoFilamentExtruderSchematic.sch (KiCad schematic (older format))
At the start: 18 parts, among them K1 ADW11, M1 Motor_DC, M2 Fan, M3 Motor_DC, Q1 Q_PMOS_GDS, U1 AC, U10 ARDUINO_MKR_485_SHIELD, U2 120ACV_24VDC, U3 24V_12V, U4 SpeedController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

Commit message: Updated extruder PCB for latest KiCad version.
Parts:
- D1, D2, D3, D4: symbol Device:D -> ValpoFilamentExtruderSchematic-rescue:D-Device
- K1: symbol Relay:ADW11 -> ValpoFilamentExtruderSchematic-rescue:ADW11-Relay
- M1, M3: symbol Motor:Motor_DC -> ValpoFilamentExtruderSchematic-rescue:Motor_DC-Motor
- M2: symbol Motor:Fan -> ValpoFilamentExtruderSchematic-rescue:Fan-Motor
- Q1: symbol Device:Q_PMOS_GDS -> ValpoFilamentExtruderSchematic-rescue:Q_PMOS_GDS-Device
- TH1: symbol Sensor_Temperature:PT100 -> ValpoFilamentExtruderSchematic-rescue:PT100-Sensor_Temperature
Connections:
- new net: U10.~ (TX), U6.~ (Th2Out)
Changed lines of the file:
@@
 $EndDescr
 $Comp
-L Sensor_Temperature:PT100 TH1
+L ValpoFilamentExtruderSchematic-rescue:PT100-Sensor_Temperature TH1
 U 1 1 5F891ED8
 P 1950 1700
@@
 	4850 6800 5250 6800
 $Comp
-L power:+5V #PWR010
+L ValpoFilamentExtruderSchematic-rescue:+5V-power #PWR010
 U 1 1 5F8A6013
 P 5250 6800
@@
 $EndComp
 $Comp
-L power:+24V #PWR07
+L ValpoFilamentExtruderSchematic-rescue:+24V-power #PWR07
 U 1 1 5F8A6838
 P 3500 6600
@@
 	2550 6600 2650 6600
 $Comp
-L Motor:Motor_DC M1
+L ValpoFilamentExtruderSchematic-rescue:Motor_DC-Motor M1
 U 1 1 5F8662F0
 P 4750 4650
@@
 $EndComp
 $Comp
-L power:+24V #PWR03
+L ValpoFilamentExtruderSchematic-rescue:+24V-power #PWR03
 U 1 1 5F8C9495
 P 1950 4200
@@
 $EndComp
 $Comp
-L power:GND #PWR04
+L ValpoFilamentExtruderSchematic-rescue:GND-power #PWR04
 U 1 1 5F8C9996
 P 2950 5150
@@
 	2700 1950 3300 1950
 $Comp
-L power:GND #PWR09
+L ValpoFilamentExtruderSchematic-rescue:GND-power #PWR09
 U 1 1 5F8D9C8A
 P 3300 1750
@@
 $EndComp
 $Comp
-L power:GND #PWR025
+L ValpoFilamentExtruderSchematic-rescue:GND-power #PWR025
 U 1 1 5F8D03BA
 P 4850 6500
@@
 $EndComp
 $Comp
-L power:GND #PWR022
+L ValpoFilamentExtruderSchematic-rescue:GND-power #PWR022
 U 1 1 5F8D08A6
 P 3600 6700
@@
 RX
 $Comp
-L power:GND #PWR024
+L ValpoFilamentExtruderSchematic-rescue:GND-power #PWR024
 U 1 1 5F8DD893
 P 3650 3200
@@
 $EndComp
 $Comp
-L power:+5V #PWR023
+L ValpoFilamentExtruderSchematic-rescue:+5V-power #PWR023
 U 1 1 5F8DD343
 P 3650 3000
@@
 	4750 2050 4750 2350
 $Comp
-L Relay:ADW11 K1
+L ValpoFilamentExtruderSchematic-rescue:ADW11-Relay K1
 U 1 1 5F904063
 P 5400 1800
@@
 Not Implemented
 $Comp
-L Device:D D1
+L ValpoFilamentExtruderSchematic-rescue:D-Device D1
 U 1 1 607F6406
 P 3850 4200
@@
 $EndComp
 $Comp
-L Device:D D2
+L ValpoFilamentExtruderSchematic-rescue:D-Device D2
 U 1 1 607F6D4D
 P 4200 4500
@@
 	2550 6650 2550 6600
 $Comp
-L Motor:Fan M2
+L ValpoFilamentExtruderSchematic-rescue:Fan-Motor M2
 U 1 1 6082F6E1
 P 7550 5150
@@
 	7550 4600 7550 4850
 $Comp
-L Motor:Motor_DC M3
+L ValpoFilamentExtruderSchematic-rescue:Motor_DC-Motor M3
 U 1 1 608327A3
 P 10450 4550
@@
 $EndComp
 $Comp
-L Device:D D4
+L ValpoFilamentExtruderSchematic-rescue:D-Device D4
 U 1 1 60832C69
 P 9800 4600
@@
 $EndComp
 $Comp
-L Device:D D3
+L ValpoFilamentExtruderSchematic-rescue:D-Device D3
 U 1 1 60832F86
 P 9350 4900
@@
 $EndComp
 $Comp
-L Device:Q_PMOS_GDS Q1
+L ValpoFilamentExtruderSchematic-rescue:Q_PMOS_GDS-Device Q1
 U 1 1 60833471
 P 8900 5250
@@
 SpoilerSignalPCB
 $Comp
-L power:GND #PWR05
+L ValpoFilamentExtruderSchematic-rescue:GND-power #PWR05
 U 1 1 608367FD
 P 9000 5650
@@
 Connection ~ 9800 4900
 $Comp
-L power:+24V #PWR06
+L ValpoFilamentExtruderSchematic-rescue:+24V-power #PWR06
 U 1 1 6083A8BB
 P 9300 4200
@@
 Connection ~ 9800 4200
 $Comp
-L power:+12V #PWR011
+L ValpoFilamentExtruderSchematic-rescue:+12V-power #PWR011
 U 1 1 6083BC6F
 P 9850 1150
@@
 $EndComp
 $Comp
-L power:+5V #PWR012
+L ValpoFilamentExtruderSchematic-rescue:+5V-power #PWR012
 U 1 1 6083C212
 P 9850 1400
@@
 $EndComp
 $Comp
-L power:GND #PWR08
+L ValpoFilamentExtruderSchematic-rescue:GND-power #PWR08
 U 1 1 6083C58D
 P 9800 1750
@@
 	4150 6650 3600 6650
 $Comp
-L power:GND #PWR01
+L ValpoFilamentExtruderSchematic-rescue:GND-power #PWR01
 U 1 1 607EA678
 P 5100 5750
@@
 $EndComp
 $Comp
-L power:+24V #PWR02
+L ValpoFilamentExtruderSchematic-rescue:+24V-power #PWR02
 U 1 1 607EA9FD
 P 5350 6050
